Commit message: Fix errores en el urdf

File: urdf/HoverRobot.urdf (robot description, URDF)
Before this commit: robot HoverRobot, 1 links, 0 joints
Links:
- link base_link: mass 4.6233 -> None

Commit message: Agrego base_footprint

File: urdf/HoverRobot.urdf (robot description, URDF)
Before this commit: robot HoverRobot, 1 links, 0 joints
Links:
- added link base_footprint
Joints:
- added joint base_footprint_to_base_link: type fixed, parent base_footprint, child base_link, origin xyz=0 0 0.48 rpy=0 0 0
